File: PowerSource.sch (KiCad schematic (older format))
At the start: 11 parts, among them U3 MC7805_TO252-3(DPACK), U4 TLV2217_TO252-3

Commit message: Se Organiza conexiones de alimentacion con elementos de la biblioteca power, se quitan algunas etiquetas y se coloca la fuente en hoja principal
Parts:
- removed C1: 0.1uF, symbol Device:CP
- removed C2: 22uF, symbol Device:CP
- removed C3: 1uF, symbol Device:CP
- removed C4: 10uF, symbol Device:CP
- removed D1: D, symbol Device:D
- removed D2: D_TVS_DESD5V0S1BA-7DITR-ND, symbol Device:D_TVS
- removed D3: D_TVS_3V3, symbol Device:D_TVS
- removed D6: LED, symbol Device:LED
- removed R12: 330, symbol Device:R
- removed U3: MC7805_TO252-3(DPACK), symbol J_ReguladorLinear:MC7805_TO252-3(DPACK)
- removed U4: TLV2217_TO252-3, symbol J_ReguladorLinear:TLV2217_TO252-3
