File: Microcontroller.sch (KiCad schematic (older format))
At the start: 15 parts, among them J6 Conn_01x06_Male, SW1 SW_Push, SW2 SW_Push, U2 PIC16F1934-IPT_J, Y1 Crystal

Commit message: TP Finalizado
Parts:
- C5, C6:  Part Number (none) -> 732-7748-1-ND; Part Number 732-7748-1-ND -> (none)
- C7:  Part Number (none) -> 399-1282-2-ND
- J6, JP1:  Part Number (none) -> 952-2521-ND
- R1, R2:  Part Number (none) -> P470DBTR-ND
- R3, R4, R5, R6:  Part Number (none) -> 1276-3485-2-ND
- SW1, SW2:  Part Number (none) -> 450-1804-ND; Part Number 450-1804-ND -> (none)
- U2: footprint (none) -> package_TQFP;  Part Number (none) -> PIC16F1934-I/PT-ND
- Y1:  Part Number (none) -> XC1776TR-ND
Changed lines of the file:
@@
 F 1 "Jumper_NC_Dual" H 5700 2550 50  0000 C CNN
 F 2 "Connector_PinSocket_2.54mm:PinSocket_1x03_P2.54mm_Vertical" H 5700 2200 50  0001 C CNN
-F 3 "~" H 5700 2200 50  0001 C CNN
+F 3 "https://cdn.harwin.com/pdfs/D01-992.pdf" H 5700 2200 50  0001 C CNN
+F 4 "952-2521-ND" H 5700 2200 50  0001 C CNN " Part Number"
 	1    5700 2200
 	1    0    0    -1
@@
 F 1 "Crystal" V 2555 4319 50  0000 R CNN
 F 2 "Crystal:Crystal_HC18-U_Vertical" H 2600 4450 50  0001 C CNN
-F 3 "~" H 2600 4450 50  0001 C CNN
+F 3 "~http://www.ecsxtal.com/store/pdf/CSM-3X.pdf" H 2600 4450 50  0001 C CNN
+F 4 "XC1776TR-ND" H 2600 4450 50  0001 C CNN " Part Number"
 	1    2600 4450
 	0    -1   -1   0
@@
 F 1 "22pF" V 2561 4250 50  0000 C CNN
 F 2 "Capacitor_SMD:C_0603_1608Metric" H 2438 4100 50  0001 C CNN
-F 3 "~" H 2400 4250 50  0001 C CNN
-F 4 "732-7748-1-ND" V 2400 4250 50  0001 C CNN "Part Number"
+F 3 "https://content.kemet.com/datasheets/KEM_C1002_X7R_SMD.pdf" H 2400 4250 50  0001 C CNN
+F 4 "732-7748-1-ND" H 2400 4250 50  0001 C CNN " Part Number"
 	1    2400 4250
 	0    -1   -1   0
@@
 F 1 "22pF" V 2561 4700 50  0000 C CNN
 F 2 "Capacitor_SMD:C_0603_1608Metric" H 2438 4550 50  0001 C CNN
-F 3 "~" H 2400 4700 50  0001 C CNN
-F 4 "732-7748-1-ND" V 2400 4700 50  0001 C CNN "Part Number"
+F 3 "https://content.kemet.com/datasheets/KEM_C1002_X7R_SMD.pdf" H 2400 4700 50  0001 C CNN
+F 4 "732-7748-1-ND" H 2400 4700 50  0001 C CNN " Part Number"
 	1    2400 4700
 	0    -1   -1   0
@@
 F 1 "SW_Push" H 9350 5594 50  0000 C CNN
 F 2 "Button_Switch_THT:SW_PUSH_6mm_H5mm" H 9350 5600 50  0001 C CNN
-F 3 "~" H 9350 5600 50  0001 C CNN
-F 4 "450-1804-ND" H 9350 5400 50  0001 C CNN "Part Number"
+F 3 "https://www.te.com/commerce/DocumentDelivery/DDEController?Action=srchrtrv&DocNm=1825910&DocType=Customer+Drawing&DocLang=English" H 9350 5600 50  0001 C CNN
+F 4 "450-1804-ND" H 9350 5400 50  0001 C CNN " Part Number"
 	1    9350 5400
 	1    0    0    -1
@@
 F 1 "10K" H 9920 5155 50  0000 L CNN
 F 2 "Resistor_SMD:R_0603_1608Metric_Pad1.05x0.95mm_HandSolder" V 9780 5200 50  0001 C CNN
-F 3 "~" H 9850 5200 50  0001 C CNN
+F 3 "http://www.samsungsem.com/kr/support/product-search/chip-resistor/__icsFiles/afieldfile/2019/01/21/RC_Spec_Sheet(1901).pdf" H 9850 5200 50  0001 C CNN
+F 4 "1276-3485-2-ND" H 9850 5200 50  0001 C CNN " Part Number"
 	1    9850 5200
 	1    0    0    -1
@@
 F 1 "0.1uF" V 6039 2550 50  0000 C CNN
 F 2 "Capacitor_SMD:C_0603_1608Metric" H 6238 2400 50  0001 C CNN
-F 3 "~" H 6200 2550 50  0001 C CNN
+F 3 "https://content.kemet.com/datasheets/KEM_C1002_X7R_SMD.pdf" H 6200 2550 50  0001 C CNN
 F 4 "732-7939-1-ND" V 6200 2550 50  0001 C CNN "Part Number"
+F 5 "399-1282-2-ND" H 6200 2550 50  0001 C CNN " Part Number"
 	1    6200 2550
 	0    1    1    0
@@
 F 1 "DNP-10K" H 9920 5505 50  0000 L CNN
 F 2 "Resistor_SMD:R_0603_1608Metric_Pad1.05x0.95mm_HandSolder" V 9780 5550 50  0001 C CNN
-F 3 "~" H 9850 5550 50  0001 C CNN
+F 3 "http://www.samsungsem.com/kr/support/product-search/chip-resistor/__icsFiles/afieldfile/2019/01/21/RC_Spec_Sheet(1901).pdf" H 9850 5550 50  0001 C CNN
+F 4 "1276-3485-2-ND" H 9850 5550 50  0001 C CNN " Part Number"
 	1    9850 5550
 	1    0    0    -1
@@
 F 1 "SW_Push" H 9350 1744 50  0000 C CNN
 F 2 "Button_Switch_THT:SW_PUSH_6mm_H5mm" H 9350 1750 50  0001 C CNN
-F 3 "~" H 9350 1750 50  0001 C CNN
-F 4 "450-1804-ND" H 9350 1550 50  0001 C CNN "Part Number"
+F 3 "https://www.te.com/commerce/DocumentDelivery/DDEController?Action=srchrtrv&DocNm=1825910&DocType=Customer+Drawing&DocLang=English" H 9350 1750 50  0001 C CNN
+F 4 "450-1804-ND" H 9350 1550 50  0001 C CNN " Part Number"
 	1    9350 1550
 	1    0    0    -1
@@
 F 1 "10K" H 9920 1305 50  0000 L CNN
 F 2 "Resistor_SMD:R_0603_1608Metric_Pad1.05x0.95mm_HandSolder" V 9780 1350 50  0001 C CNN
-F 3 "~" H 9850 1350 50  0001 C CNN
+F 3 "http://www.samsungsem.com/kr/support/product-search/chip-resistor/__icsFiles/afieldfile/2019/01/21/RC_Spec_Sheet(1901).pdf" H 9850 1350 50  0001 C CNN
+F 4 "1276-3485-2-ND" H 9850 1350 50  0001 C CNN " Part Number"
 	1    9850 1350
 	1    0    0    -1
@@
 F 1 "DNP-10K" H 9920 1655 50  0000 L CNN
 F 2 "Resistor_SMD:R_0603_1608Metric_Pad1.05x0.95mm_HandSolder" V 9780 1700 50  0001 C CNN
-F 3 "~" H 9850 1700 50  0001 C CNN
+F 3 "http://www.samsungsem.com/kr/support/product-search/chip-resistor/__icsFiles/afieldfile/2019/01/21/RC_Spec_Sheet(1901).pdf" H 9850 1700 50  0001 C CNN
+F 4 "1276-3485-2-ND" H 9850 1700 50  0001 C CNN " Part Number"
 	1    9850 1700
 	1    0    0    -1
@@
 F 1 "470" V 8050 3700 50  0000 L CNN
 F 2 "Resistor_SMD:R_0603_1608Metric_Pad1.05x0.95mm_HandSolder" V 7880 3900 50  0001 C CNN
-F 3 "~" H 7950 3900 50  0001 C CNN
+F 3 "https://industrial.panasonic.com/cdbs/www-data/pdf/RDM0000/AOA0000C307.pdf" H 7950 3900 50  0001 C CNN
+F 4 "P470DBTR-ND" H 7950 3900 50  0001 C CNN " Part Number"
 	1    7950 3900
 	0    -1   -1   0
@@
 F 1 "470" V 7850 3800 50  0000 L CNN
 F 2 "Resistor_SMD:R_0603_1608Metric_Pad1.05x0.95mm_HandSolder" V 7880 4000 50  0001 C CNN
-F 3 "~" H 7950 4000 50  0001 C CNN
+F 3 "https://industrial.panasonic.com/cdbs/www-data/pdf/RDM0000/AOA0000C307.pdf" H 7950 4000 50  0001 C CNN
+F 4 "P470DBTR-ND" H 7950 4000 50  0001 C CNN " Part Number"
 	1    7950 4000
 	0    -1   -1   0
@@
 F 1 "Conn_01x06_Male" H 2300 900 50  0000 R CNN
 F 2 "Connector_PinSocket_2.54mm:PinSocket_1x06_P2.54mm_Vertical" H 1700 1450 50  0001 C CNN
-F 3 "~" H 1700 1450 50  0001 C CNN
+F 3 "https://cdn.harwin.com/pdfs/D01-992.pdf" H 1700 1450 50  0001 C CNN
+F 4 "952-2521-ND" H 1700 1450 50  0001 C CNN " Part Number"
 	1    1700 1450
 	1    0    0    -1
@@
 F 0 "U2" H 7300 5700 50  0000 C CNN
 F 1 "PIC16F1934-IPT_J" H 4400 5700 50  0000 C CNN
-F 2 "" H 5700 4400 50  0001 C CNN
+F 2 "package_TQFP" H 5700 4400 50  0001 C CNN
 F 3 "http://ww1.microchip.com/downloads/en/DeviceDoc/41364E.pdf" H 5700 4400 50  0001 C CNN
+F 4 "PIC16F1934-I/PT-ND" H 5700 4400 50  0001 C CNN " Part Number"
 	1    5700 4400
 	1    0    0    -1
