File: SensorsIO.sch (KiCad schematic (older format))
At the start: 11 parts, among them J3 Conn_01x10_Male, J4 Conn_01x04_Male, J5 Conn_01x04_Male

Commit message: TP Finalizado
Parts:
- D4:  Part Number (none) -> 160-1446-6-ND
- D5:  Part Number (none) -> 516-1778-6-ND; Part Number 516-1778-6-ND -> (none)
- J3, J4, J5:  Part Number (none) -> 952-2521-ND
- R10, R7, R8, R9:  Part Number (none) -> RHM330AZCT-ND
- R11:  Part Number (none) -> P1.00KHDKR-ND
- RV1:  Part Number (none) -> 987-1305-ND; Part Number 987-1305-ND -> (none)
Changed lines of the file:
@@
 F 1 "330" H 5870 3605 50  0000 L CNN
 F 2 "Resistor_SMD:R_0603_1608Metric_Pad1.05x0.95mm_HandSolder" V 5730 3650 50  0001 C CNN
-F 3 "~" H 5800 3650 50  0001 C CNN
+F 3 "https://www.rohm.com/datasheet/KTR03EZPF/ktr-e" H 5800 3650 50  0001 C CNN
+F 4 "RHM330AZCT-ND" H 5800 3650 50  0001 C CNN " Part Number"
 	1    5800 3650
 	1    0    0    -1
@@
 F 1 "LED" V 5748 3933 50  0000 R CNN
 F 2 "LED_SMD:LED_0603_1608Metric_Castellated" H 5800 4050 50  0001 C CNN
-F 3 "~" H 5800 4050 50  0001 C CNN
+F 3 "http://optoelectronics.liteon.com/upload/download/DS22-2000-228/LTST-C191KGKT.PDF" H 5800 4050 50  0001 C CNN
 F 4 "160-1447-1-ND" V 5800 4050 50  0001 C CNN "Part number"
+F 5 "160-1446-6-ND" H 5800 4050 50  0001 C CNN " Part Number"
 	1    5800 4050
 	0    -1   -1   0
@@
 F 1 "Conn_01x04_Male" V 3300 5200 50  0000 R CNN
 F 2 "Connector_PinSocket_2.54mm:PinSocket_1x04_P2.54mm_Vertical" H 3550 5000 50  0001 C CNN
-F 3 "~" H 3550 5000 50  0001 C CNN
+F 3 "https://cdn.harwin.com/pdfs/D01-992.pdf" H 3550 5000 50  0001 C CNN
+F 4 "952-2521-ND" H 3550 5000 50  0001 C CNN " Part Number"
 	1    3550 5000
 	-1   0    0    1
@@
 F 1 "Conn_01x04_Male" V 3650 3900 50  0000 R CNN
 F 2 "Connector_PinSocket_2.54mm:PinSocket_1x04_P2.54mm_Vertical" H 3900 3500 50  0001 C CNN
-F 3 "~" H 3900 3500 50  0001 C CNN
+F 3 "https://cdn.harwin.com/pdfs/D01-992.pdf" H 3900 3500 50  0001 C CNN
+F 4 "952-2521-ND" H 3900 3500 50  0001 C CNN " Part Number"
 	1    3900 3500
 	-1   0    0    1
@@
 F 1 "330" V 7050 3500 50  0000 L CNN
 F 2 "Resistor_SMD:R_0603_1608Metric_Pad1.05x0.95mm_HandSolder" V 6880 3700 50  0001 C CNN
-F 3 "~" H 6950 3700 50  0001 C CNN
+F 3 "https://www.rohm.com/datasheet/KTR03EZPF/ktr-e" H 6950 3700 50  0001 C CNN
+F 4 "RHM330AZCT-ND" H 6950 3700 50  0001 C CNN " Part Number"
 	1    6950 3700
 	1    0    0    -1
@@
 F 1 "330" V 6650 3500 50  0000 L CNN
 F 2 "Resistor_SMD:R_0603_1608Metric_Pad1.05x0.95mm_HandSolder" V 6680 3700 50  0001 C CNN
-F 3 "~" H 6750 3700 50  0001 C CNN
+F 3 "https://www.rohm.com/datasheet/KTR03EZPF/ktr-e" H 6750 3700 50  0001 C CNN
+F 4 "RHM330AZCT-ND" H 6750 3700 50  0001 C CNN " Part Number"
 	1    6750 3700
 	1    0    0    -1
@@
 F 1 "330" V 6450 3500 50  0000 L CNN
 F 2 "Resistor_SMD:R_0603_1608Metric_Pad1.05x0.95mm_HandSolder" V 6480 3700 50  0001 C CNN
-F 3 "~" H 6550 3700 50  0001 C CNN
+F 3 "https://www.rohm.com/datasheet/KTR03EZPF/ktr-e" H 6550 3700 50  0001 C CNN
+F 4 "RHM330AZCT-ND" H 6550 3700 50  0001 C CNN " Part Number"
 	1    6550 3700
 	1    0    0    -1
@@
 F 1 "Conn_01x10_Male" V 3650 2800 50  0000 R CNN
 F 2 "Connector_PinSocket_2.54mm:PinSocket_1x10_P2.54mm_Vertical" H 3900 2500 50  0001 C CNN
-F 3 "~" H 3900 2500 50  0001 C CNN
+F 3 "https://cdn.harwin.com/pdfs/D01-992.pdf" H 3900 2500 50  0001 C CNN
+F 4 "952-2521-ND" H 3900 2500 50  0001 C CNN " Part Number"
 	1    3900 2500
 	-1   0    0    -1
@@
 F 1 "1K" H 8570 4305 50  0000 L CNN
 F 2 "Resistor_SMD:R_0603_1608Metric_Pad1.05x0.95mm_HandSolder" V 8430 4350 50  0001 C CNN
-F 3 "~" H 8500 4350 50  0001 C CNN
+F 3 "https://industrial.panasonic.com/cdbs/www-data/pdf/RDA0000/AOA0000C304.pdf" H 8500 4350 50  0001 C CNN
+F 4 "P1.00KHDKR-ND" H 8500 4350 50  0001 C CNN " Part Number"
 	1    8500 4350
 	1    0    0    -1
@@
 F 1 "10K" H 8431 3855 50  0000 R CNN
 F 2 "Potentiometer_SMD:Potentiometer_ACP_CA6-VSMD_Vertical" H 8500 3900 50  0001 C CNN
-F 3 "~" H 8500 3900 50  0001 C CNN
-F 4 "987-1305-ND" H 8500 3900 50  0001 C CNN "Part Number"
+F 3 "https://www.ttelectronics.com/TTElectronics/media/ProductFiles/Potentiometers/Datasheets/P160.pdf" H 8500 3900 50  0001 C CNN
+F 4 "987-1305-ND" H 8500 3900 50  0001 C CNN " Part Number"
 	1    8500 3900
 	1    0    0    -1
@@
 F 1 "LED_CRGB" V 6705 3920 50  0000 R CNN
 F 2 "LED_SMD:LED_RGB_1210" H 6750 4200 50  0001 C CNN
-F 3 "~" H 6750 4200 50  0001 C CNN
-F 4 "	516-1778-6-ND" V 6750 4250 50  0001 C CNN "Part Number"
+F 3 "https://docs.broadcom.com/docs/AV02-0610EN" H 6750 4200 50  0001 C CNN
+F 4 "	516-1778-6-ND" H 6750 4250 50  0001 C CNN " Part Number"
 	1    6750 4250
 	0    -1   -1   0
