File: TPDSI_1.kicad_pcb (KiCad board)
At the start: 2 copper layers, 85 x 62.5 mm, 63 parts, among them J1 Conn_01x02_Male, J2 Conn_01x02_Male, J3 Conn_01x10_Male, J4 Conn_01x04_Male, J5 Conn_01x04_Male, J6 Conn_01x06_Male, J7 Screw_Terminal_01x02, Q1 Q_NPN_BCE, Q2 Q_NPN_BCE, SW1 SW_Push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

Commit message: TP Finalizado
Other:
- board text added: "*Colocar tented a las vias en la fabricación *Terminación HASL *Fabricante criterios dimensión : https://www.colcircuitos.com/wp-content/uploads/2017/08/ REQUERIMIENTOS-MINIMOS-FE-2017.pdf"
- board text added: "FR4 -1.6cm -35micras"
- board text removed: "*Colocar tented a las vias en la fabricación *Terminación HASL *Fabricante criterios dimención : https://www.colcircuitos.com/wp-content/uploads/2017/08/REQUERIMIENTOS-MINIMOS-FE-2017.pdf"
Changed lines of the file:
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@@
   (general
     (thickness 1.6)
-    (drawings 45)
+    (drawings 46)
     (tracks 763)
     (zones 0)
@@
     (0 F.Cu signal)
     (31 B.Cu signal)
-    (32 B.Adhes user)
-    (33 F.Adhes user)
-    (34 B.Paste user)
-    (35 F.Paste user)
+    (32 B.Adhes user hide)
+    (33 F.Adhes user hide)
+    (34 B.Paste user hide)
+    (35 F.Paste user hide)
     (36 B.SilkS user)
     (37 F.SilkS user)
@@
     )
   )
+  (gr_text "FR4 -1.6cm -35micras" (at 29.5 68.468) (layer Eco1.User)
+    (effects (font (size 1 1) (thickness 0.15)))
+  )
   (gr_text "POT ANG" (at 138.176 120.65) (layer F.SilkS)
     (effects (font (size 1 1) (thickness 0.15)))
@@
   (gr_line (start 192 61.5) (end 192 124) (layer Edge.Cuts) (width 0.05))
   (gr_line (start 107 61.5) (end 192 61.5) (layer Edge.Cuts) (width 0.05))
-  (gr_text "*Colocar tented a las vias en la fabricación\n*Terminación HASL\n*Fabricante criterios dimención :\n https://www.colcircuitos.com/wp-content/uploads/2017/08/REQUERIMIENTOS-MINIMOS-FE-2017.pdf" (at 20.038 87) (layer Eco1.User)
+  (gr_text "*Colocar tented a las vias en la fabricación\n*Terminación HASL\n*Fabricante criterios dimensión :\n https://www.colcircuitos.com/wp-content/uploads/2017/08/\n REQUERIMIENTOS-MINIMOS-FE-2017.pdf" (at 20.038 87) (layer Eco1.User)
     (effects (font (size 1 1) (thickness 0.15)) (justify left))
   )
