File: TPDSI_1.sch (KiCad schematic (older format))
At the start: 22 parts, among them J1 Conn_01x02_Male, J2 Conn_01x02_Male, J7 Screw_Terminal_01x02, U3 MC7805_TO252-3(DPACK), U4 TLV2217_TO252-3

Commit message: Se agregan cosas obligatorias por norma y algunas sugerencias por el docente
Parts:
- C4: Part Number (none) -> 399-16038-1-ND; Part number 399-16038-1-ND -> (none)
- D1: PArt Number 1N4148W-FDICT-ND -> (none); Part Number (none) -> 1N4148W-FDICT-ND
Changed lines of the file:
@@
 F 2 "Capacitor_Tantalum_SMD:CP_EIA-7343-20_Kemet-V" H 6438 1450 50  0001 C CNN
 F 3 "~" H 6400 1600 50  0001 C CNN
-F 4 "399-16038-1-ND" H 6400 1600 50  0001 C CNN "Part number"
+F 4 "399-16038-1-ND" H 6400 1600 50  0001 C CNN "Part Number"
 	1    6400 1600
 	1    0    0    -1
@@
 F 2 "Diode_SMD:D_SOD-123" H 3300 1200 50  0001 C CNN
 F 3 "~" H 3300 1200 50  0001 C CNN
-F 4 "1N4148W-FDICT-ND" H 3300 1200 50  0001 C CNN "PArt Number"
+F 4 "1N4148W-FDICT-ND" H 3300 1200 50  0001 C CNN "Part Number"
 	1    3300 1200
 	-1   0    0    -1
@@
 Wire Wire Line
 	4950 1750 4950 1850
-Wire Wire Line
-	4950 1850 4900 1850
 Connection ~ 4650 1850
 Wire Wire Line
@@
 $EndComp
 Wire Wire Line
-	4900 1900 4900 1850
-Connection ~ 4900 1850
-Wire Wire Line
-	4900 1850 4650 1850
-Wire Wire Line
 	4500 1200 4650 1200
 Wire Wire Line
@@
 Wire Bus Line
 	4050 4250 4050 5250
+Wire Wire Line
+	4650 1850 4950 1850
 $EndSCHEMATC

Commit message: TP Finalizado
Parts:
- C1:  Part Number (none) -> 718-1117-2-ND; Part Number 399-14253-2-ND -> ..
- C2:  Part Number (none) -> P16517DKR-ND; Part Number P16517DKR-ND -> (none)
- C3:  Part Number (none) -> 718-1117-2-ND; Part Number (none) -> ..
- C4:  Part Number (none) -> 399-16038-1-ND; Part Number 399-16038-1-ND -> (none)
- D1:  Part Number (none) -> 1N4148W-FDICT-ND; Part Number 1N4148W-FDICT-ND -> (none)
- D2:  Part Number (none) -> 160-1446-6-ND
- D3:  Part Number (none) -> 497-2999-2-ND
- D6:  Part Number (none) -> 641-1985-1-ND; Part Number 641-1985-1-ND -> (none)
- FID1, FID2, FID3, FID4, H1, H2, H3, H4:  Part Number (none) -> N/A
- J1, J2:  Part Number (none) -> 952-2521-ND
- J7:  Part Number (none) -> ED1613-ND
- R12:  Part Number (none) -> RHM330AZCT-ND
Changed lines of the file:
@@
 F 1 "1uF" H 3918 1555 50  0000 L CNN
 F 2 "Capacitor_Tantalum_SMD:CP_EIA-3528-21_Kemet-B" H 3838 1450 50  0001 C CNN
-F 3 "~" H 3800 1600 50  0001 C CNN
-F 4 "	399-14253-2-ND" H 3800 1600 50  0001 C CNN "Part Number"
+F 3 "https://content.kemet.com/datasheets/KEM_C1002_X7R_SMD.pdf" H 3800 1600 50  0001 C CNN
+F 4 ".." H 3800 1600 50  0001 C CNN "Part Number"
+F 5 "718-1117-2-ND" H 3800 1600 50  0001 C CNN " Part Number"
 	1    3800 1600
 	1    0    0    -1
@@
 F 1 "1uF" H 5568 1555 50  0000 L CNN
 F 2 "Capacitor_Tantalum_SMD:CP_EIA-3528-21_Kemet-B" H 5488 1450 50  0001 C CNN
-F 3 "~" H 5450 1600 50  0001 C CNN
+F 3 "https://content.kemet.com/datasheets/KEM_C1002_X7R_SMD.pdf" H 5450 1600 50  0001 C CNN
+F 4 ".." H 5450 1600 50  0001 C CNN "Part Number"
+F 5 "718-1117-2-ND" H 5450 1600 50  0001 C CNN " Part Number"
 	1    5450 1600
 	1    0    0    -1
@@
 F 1 "10uF" H 6518 1555 50  0000 L CNN
 F 2 "Capacitor_Tantalum_SMD:CP_EIA-7343-20_Kemet-V" H 6438 1450 50  0001 C CNN
-F 3 "~" H 6400 1600 50  0001 C CNN
-F 4 "399-16038-1-ND" H 6400 1600 50  0001 C CNN "Part Number"
+F 3 "https://content.kemet.com/datasheets/KEM_C1002_X7R_SMD.pdf" H 6400 1600 50  0001 C CNN
+F 4 "399-16038-1-ND" H 6400 1600 50  0001 C CNN " Part Number"
 	1    6400 1600
 	1    0    0    -1
@@
 F 1 "1n4148" H 3300 1325 50  0000 C CNN
 F 2 "Diode_SMD:D_SOD-123" H 3300 1200 50  0001 C CNN
-F 3 "~" H 3300 1200 50  0001 C CNN
-F 4 "1N4148W-FDICT-ND" H 3300 1200 50  0001 C CNN "Part Number"
+F 3 "https://www.diodes.com/assets/Datasheets/ds30086.pdf" H 3300 1200 50  0001 C CNN
+F 4 "1N4148W-FDICT-ND" H 3300 1200 50  0001 C CNN " Part Number"
 	1    3300 1200
 	-1   0    0    -1
@@
 F 1 "D_TVS_3V3" H 6750 1900 50  0000 L CNN
 F 2 "Diode_SMD:D_SOD-123" H 6900 1600 50  0001 C CNN
-F 3 "~" H 6900 1600 50  0001 C CNN
-F 4 "641-1985-1-ND" V 6900 1600 50  0001 C CNN "Part Number"
+F 3 "http://www.comchiptech.com/admin/files/product/TV02W-G%20series%20RevE.pdf" H 6900 1600 50  0001 C CNN
+F 4 "641-1985-1-ND" H 6900 1600 50  0001 C CNN " Part Number"
 	1    6900 1600
 	0    1    1    0
@@
 F 1 "LED" V 3448 1633 50  0000 R CNN
 F 2 "LED_SMD:LED_0603_1608Metric_Castellated" H 3500 1750 50  0001 C CNN
-F 3 "~" H 3500 1750 50  0001 C CNN
+F 3 "http://optoelectronics.liteon.com/upload/download/DS22-2000-228/LTST-C191KGKT.PDF" H 3500 1750 50  0001 C CNN
 F 4 "	160-1446-6-ND" V 3500 1750 50  0001 C CNN "PArt Number"
+F 5 "160-1446-6-ND" H 3500 1750 50  0001 C CNN " Part Number"
 	1    3500 1750
 	0    -1   -1   0
@@
 F 1 "330" H 3570 1305 50  0000 L CNN
 F 2 "Resistor_SMD:R_0603_1608Metric_Pad1.05x0.95mm_HandSolder" V 3430 1350 50  0001 C CNN
-F 3 "~" H 3500 1350 50  0001 C CNN
+F 3 "https://www.rohm.com/datasheet/KTR03EZPF/ktr-e" H 3500 1350 50  0001 C CNN
+F 4 "RHM330AZCT-ND" H 3500 1350 50  0001 C CNN " Part Number"
 	1    3500 1350
 	1    0    0    -1
@@
 F 1 "D_TVS_DESD5V0S1BA-7DITR-ND" V 5550 800 50  0001 L CNN
 F 2 "Diode_SMD:D_SOD-123" H 4950 1600 50  0001 C CNN
-F 3 "~" H 4950 1600 50  0001 C CNN
+F 3 "https://www.st.com/content/ccc/resource/technical/document/datasheet/ff/c0/80/cc/19/4c/45/af/CD00001333.pdf/files/CD00001333.pdf/_jcr_content/translations/en.CD00001333.pdf" H 4950 1600 50  0001 C CNN
+F 4 "497-2999-2-ND" H 4950 1600 50  0001 C CNN " Part Number"
 	1    4950 1600
 	0    1    1    0
@@
 F 1 "Conn_01x02_Male" H 7322 3823 50  0000 R CNN
 F 2 "Connector_PinSocket_2.54mm:PinSocket_1x02_P2.54mm_Vertical" H 7350 3850 50  0001 C CNN
-F 3 "~" H 7350 3850 50  0001 C CNN
+F 3 "https://cdn.harwin.com/pdfs/D01-992.pdf" H 7350 3850 50  0001 C CNN
+F 4 "952-2521-ND" H 7350 3850 50  0001 C CNN " Part Number"
 	1    7350 3850
 	-1   0    0    1
@@
 F 1 "Conn_01x02_Male" H 7322 4073 50  0000 R CNN
 F 2 "Connector_PinSocket_2.54mm:PinSocket_1x02_P2.54mm_Vertical" H 7350 4100 50  0001 C CNN
-F 3 "~" H 7350 4100 50  0001 C CNN
+F 3 "https://cdn.harwin.com/pdfs/D01-992.pdf" H 7350 4100 50  0001 C CNN
+F 4 "952-2521-ND" H 7350 4100 50  0001 C CNN " Part Number"
 	1    7350 4100
 	-1   0    0    1
@@
 F 1 "Screw_Terminal_01x02" V 2950 1350 50  0000 C CNN
 F 2 "TerminalBlock:TerminalBlock_bornier-2_P5.08mm" H 2800 1300 50  0001 C CNN
-F 3 "~" H 2800 1300 50  0001 C CNN
+F 3 "http://www.on-shore.com/wp-content/uploads/2015/09/ed130ds.pdf" H 2800 1300 50  0001 C CNN
+F 4 "ED1613-ND" H 2800 1300 50  0001 C CNN " Part Number"
 	1    2800 1300
 	-1   0    0    1
@@
 F 1 "MountingHole" H 10300 1755 50  0000 L CNN
 F 2 "MountingHole:MountingHole_3.2mm_M3" H 10200 1800 50  0001 C CNN
-F 3 "~" H 10200 1800 50  0001 C CNN
+F 3 "N/A" H 10200 1800 50  0001 C CNN
+F 4 "N/A" H 10200 1800 50  0001 C CNN " Part Number"
 	1    10200 1800
 	1    0    0    -1
@@
 F 1 "MountingHole" H 10300 2055 50  0000 L CNN
 F 2 "MountingHole:MountingHole_3.2mm_M3" H 10200 2100 50  0001 C CNN
-F 3 "~" H 10200 2100 50  0001 C CNN
+F 3 "N/A" H 10200 2100 50  0001 C CNN
+F 4 "N/A" H 10200 2100 50  0001 C CNN " Part Number"
 	1    10200 2100
 	1    0    0    -1
@@
 F 1 "MountingHole" H 10300 2355 50  0000 L CNN
 F 2 "MountingHole:MountingHole_3.2mm_M3" H 10200 2400 50  0001 C CNN
-F 3 "~" H 10200 2400 50  0001 C CNN
+F 3 "N/A" H 10200 2400 50  0001 C CNN
+F 4 "N/A" H 10200 2400 50  0001 C CNN " Part Number"
 	1    10200 2400
 	1    0    0    -1
@@
 F 1 "MountingHole" H 10300 2605 50  0000 L CNN
 F 2 "MountingHole:MountingHole_3.2mm_M3" H 10200 2650 50  0001 C CNN
-F 3 "~" H 10200 2650 50  0001 C CNN
+F 3 "N/A" H 10200 2650 50  0001 C CNN
+F 4 "N/A" H 10200 2650 50  0001 C CNN " Part Number"
 	1    10200 2650
 	1    0    0    -1
@@
 F 1 "22uF" H 4400 1500 50  0000 L CNN
 F 2 "Capacitor_Tantalum_SMD:CP_EIA-7343-20_Kemet-V" H 4688 1450 50  0001 C CNN
-F 3 "~" H 4650 1600 50  0001 C CNN
-F 4 "P16517DKR-ND" H 4650 1600 50  0001 C CNN "Part Number"
+F 3 "https://content.kemet.com/datasheets/KEM_C1002_X7R_SMD.pdf" H 4650 1600 50  0001 C CNN
+F 4 "P16517DKR-ND" H 4650 1600 50  0001 C CNN " Part Number"
 	1    4650 1600
 	1    0    0    -1
@@
 F 1 "Fiducial" H 10285 3355 50  0000 L CNN
 F 2 "Fiducial:Fiducial_1mm_Mask2mm" H 10200 3400 50  0001 C CNN
-F 3 "~" H 10200 3400 50  0001 C CNN
+F 3 "N/A" H 10200 3400 50  0001 C CNN
+F 4 "N/A" H 10200 3400 50  0001 C CNN " Part Number"
 	1    10200 3400
 	1    0    0    -1
@@
 F 1 "Fiducial" H 10285 3605 50  0000 L CNN
 F 2 "Fiducial:Fiducial_1mm_Mask2mm" H 10200 3650 50  0001 C CNN
-F 3 "~" H 10200 3650 50  0001 C CNN
+F 3 "N/A" H 10200 3650 50  0001 C CNN
+F 4 "N/A" H 10200 3650 50  0001 C CNN " Part Number"
 	1    10200 3650
 	1    0    0    -1
@@
 F 1 "Fiducial" H 10285 3855 50  0000 L CNN
 F 2 "Fiducial:Fiducial_1mm_Mask2mm" H 10200 3900 50  0001 C CNN
-F 3 "~" H 10200 3900 50  0001 C CNN
+F 3 "N/A" H 10200 3900 50  0001 C CNN
+F 4 "N/A" H 10200 3900 50  0001 C CNN " Part Number"
 	1    10200 3900
 	1    0    0    -1
@@
 F 1 "Fiducial" H 10285 3105 50  0000 L CNN
 F 2 "Fiducial:Fiducial_1mm_Mask2mm" H 10200 3150 50  0001 C CNN
-F 3 "~" H 10200 3150 50  0001 C CNN
+F 3 "N/A" H 10200 3150 50  0001 C CNN
+F 4 "N/A" H 10200 3150 50  0001 C CNN " Part Number"
 	1    10200 3150
 	1    0    0    -1
